File: hardware/control/halt/input_supply.kicad_sch (KiCad schematic)
At the start: 17 parts, among them J1 RJ45, J2 RJ45, J3 RJ45, U1 L7812, U2 L7805, U3 74HC14, U4 74HC08, U5 74HC74

Commit message: update right about freaking everything
Parts:
- removed U4: 74HC08, symbol 74xx:74HC00
- added U13: 74LS08, symbol 74xx:74LS08
Connections:
- net GND: now also U13.7 (GND)
- net halt_5v: now also U13.14 (VCC)
Changed lines of the file:
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@@
-	)
-	(symbol
-		(lib_id "74xx:74HC00")
-		(at 115.57 118.11 90)
-		(unit 5)
-		(exclude_from_sim no)
-		(in_bom yes)
-		(on_board yes)
-		(dnp no)
-		(property "Reference" "U4"
-			(at 115.57 109.22 90)
-			(effects
-				(font
-					(size 1.27 1.27)
-				)
-			)
-		)
-		(property "Value" "74HC08"
-			(at 115.57 111.76 90)
-			(effects
-				(font
-					(size 1.27 1.27)
-				)
-			)
-		)
-		(property "Footprint" ""
-			(at 115.57 118.11 0)
-			(effects
-				(font
-					(size 1.27 1.27)
-				)
-				(hide yes)
-			)
-		)
-		(property "Datasheet" "http://www.ti.com/lit/gpn/sn74hc00"
-			(at 115.57 118.11 0)
-			(effects
-				(font
-					(size 1.27 1.27)
-				)
-				(hide yes)
-			)
-		)
-		(property "Description" "quad 2-input NAND gate"
-			(at 115.57 118.11 0)
-			(effects
-				(font
-					(size 1.27 1.27)
-				)
-				(hide yes)
-			)
-		)
-		(pin "11"
-		)
-		(pin "9"
-		)
-		(pin "8"
-		)
-		(pin "12"
-		)
-		(pin "7"
-		)
-		(pin "1"
-		)
-		(pin "3"
-		)
-		(pin "2"
-		)
-		(pin "10"
-		)
-		(pin "4"
-		)
-		(pin "13"
-		)
-		(pin "5"
-		)
-		(pin "6"
-		)
-		(pin "14"
-		)
-		(instances
-			(project "base"
-				(path "/00f9de9f-6e16-4126-a022-a7b5fad77592/8b2072f1-4473-43e6-a1a2-fbe5e7e9ad6a"
-					(reference "U4")
-					(unit 5)
-				)
-			)
-			(project "hardware"
-				(path "/606d342f-174b-4504-b335-50f65aa4e733/9d9bac97-3577-4438-bb72-9616a5994fba/8b2072f1-4473-43e6-a1a2-fbe5e7e9ad6a"
-					(reference "U4")
-					(unit 5)
-				)
-			)
-		)
 	)
 	(symbol
@@
 				)
 			)
+		)
+	)
+	(symbol
+		(lib_id "74xx:74LS08")
+		(at 115.57 118.11 90)
+		(unit 5)
+		(exclude_from_sim no)
+		(in_bom yes)
+		(on_board yes)
+		(dnp no)
+		(fields_autoplaced yes)
+		(property "Reference" "U13"
+			(at 115.57 107.95 90)
+			(effects
+				(font
+					(size 1.27 1.27)
+				)
+			)
+		)
+		(property "Value" "74LS08"
+			(at 115.57 110.49 90)
+			(effects
+				(font
+					(size 1.27 1.27)
+				)
+			)
+		)
+		(property "Footprint" ""
+			(at 115.57 118.11 0)
+			(effects
+				(font
+					(size 1.27 1.27)
+				)
+				(hide yes)
+			)
+		)
+		(property "Datasheet" "http://www.ti.com/lit/gpn/sn74LS08"
+			(at 115.57 118.11 0)
+			(effects
+				(font
+					(size 1.27 1.27)
+				)
+				(hide yes)
+			)
+		)
+		(property "Description" "Quad And2"
+			(at 115.57 118.11 0)
+			(effects
+				(font
+					(size 1.27 1.27)
+				)
+				(hide yes)
+			)
+		)
+		(pin "12"
+		)
+		(pin "10"
+		)
+		(pin "8"
+		)
+		(pin "11"
+		)
+		(pin "7"
+		)
+		(pin "13"
+		)
+		(pin "6"
+		)
+		(pin "2"
+		)
+		(pin "5"
+		)
+		(pin "4"
+		)
+		(pin "1"
+		)
+		(pin "3"
+		)
+		(pin "9"
+		)
+		(pin "14"
+		)
+		(instances
+			(project ""
+				(path "/606d342f-174b-4504-b335-50f65aa4e733/9d9bac97-3577-4438-bb72-9616a5994fba/8b2072f1-4473-43e6-a1a2-fbe5e7e9ad6a"
+					(reference "U13")
+					(unit 5)
+				)
+			)
