File: hardware/control/halt/output_stage.kicad_sch (KiCad schematic)
At the start: 7 parts, among them U4 74HC08, U5 74HC74

Commit message: add progress on main drive controller and switch to hiearchical labels
Connections:
- net BUCK_OCD_OK: no longer U4.2
- new net SUPPLY_UVLO_OK: U4.2
Changed lines of the file:
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@@
 	(wire
 		(pts
-			(xy 110.49 97.79) (xy 130.81 97.79)
+			(xy 107.95 97.79) (xy 130.81 97.79)
 		)
 		(stroke
@@
 		)
 	)
-	(global_label "halt_5v"
+	(hierarchical_label "halt_5v"
 		(shape bidirectional)
 		(at 167.64 81.28 0)
-		(fields_autoplaced yes)
 		(effects
 			(font
@@
 			(justify left)
 		)
-		(property "Intersheetrefs" "${INTERSHEET_REFS}"
-			(at 178.5701 81.28 0)
-			(effects
-				(font
-					(size 1.27 1.27)
-				)
-				(justify left)
-				(hide yes)
-			)
-		)
-	)
-	(global_label "BUCK_OCD_OK"
+	)
+	(hierarchical_label "PRIMARY_OCD_OK"
+		(shape bidirectional)
+		(at 107.95 97.79 180)
+		(effects
+			(font
+				(size 1.27 1.27)
+			)
+			(justify right)
+		)
+	)
+	(hierarchical_label "BUCK_OCD_OK"
+		(shape bidirectional)
+		(at 107.95 102.87 180)
+		(effects
+			(font
+				(size 1.27 1.27)
+			)
+			(justify right)
+		)
+	)
+	(hierarchical_label "SUPPLY_UVLO_OK"
 		(shape bidirectional)
 		(at 107.95 107.95 180)
-		(fields_autoplaced yes)
-		(effects
-			(font
-				(size 1.27 1.27)
-			)
-			(justify right)
-		)
-		(property "Intersheetrefs" "${INTERSHEET_REFS}"
-			(at 90.3068 107.95 0)
-			(effects
-				(font
-					(size 1.27 1.27)
-				)
-				(justify right)
-				(hide yes)
-			)
-		)
-	)
-	(global_label "BUCK_OCD_OK"
-		(shape bidirectional)
-		(at 107.95 102.87 180)
-		(fields_autoplaced yes)
-		(effects
-			(font
-				(size 1.27 1.27)
-			)
-			(justify right)
-		)
-		(property "Intersheetrefs" "${INTERSHEET_REFS}"
-			(at 90.3068 102.87 0)
-			(effects
-				(font
-					(size 1.27 1.27)
-				)
-				(justify right)
-				(hide yes)
-			)
-		)
-	)
-	(global_label "PRIMARY_OCD_OK"
-		(shape bidirectional)
-		(at 110.49 97.79 180)
-		(fields_autoplaced yes)
-		(effects
-			(font
-				(size 1.27 1.27)
-			)
-			(justify right)
-		)
-		(property "Intersheetrefs" "${INTERSHEET_REFS}"
-			(at 89.9439 97.79 0)
-			(effects
-				(font
-					(size 1.27 1.27)
-				)
-				(justify right)
-				(hide yes)
-			)
-		)
-	)
+		(effects
+			(font
+				(size 1.27 1.27)
+			)
+			(justify right)
+		)
+	)

Commit message: update right about freaking everything
Parts:
- removed U4: 74HC08, symbol 74xx:74HC00
- added U4: 74LS08, symbol 74xx:74LS08
Connections:
- net BUCK_OCD_OK: now also U4.4
- net PRIMARY_OCD_OK: now also U4.1
- net SUPPLY_UVLO_OK: now also U4.5
- net at U5.1 (~{R}): now also U4.3
- new net: U4.2, U4.6
