File: hardware/control/inverter/base.kicad_sch (KiCad schematic)
At the start: 0 parts

Commit message: update right about freaking everything
Other:
- added sheet inverter_self_osc_feedback_pass (self_oscillation_feedback_pass.kicad_sch)
- sheet interrupt_cross_off ports: added INVERTER_RUN_STATE; removed INVERTER_FEEDBACK+, INVERTER_FEEDBACK-, INVERTER_RAW_FEEDBACK-
Changed lines of the file:
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@@
-	(wire
-		(pts
-			(xy 92.71 67.31) (xy 96.52 67.31)
-		)
-		(stroke
-			(width 0)
-			(type default)
-		)
-	)
 	(wire
 		(pts
@@
 	(wire
 		(pts
-			(xy 92.71 34.29) (xy 97.79 34.29)
-		)
-		(stroke
-			(width 0)
-			(type default)
-		)
-	)
-	(wire
-		(pts
-			(xy 40.64 77.47) (xy 59.69 77.47)
+			(xy 92.71 36.83) (xy 97.79 36.83)
+		)
+		(stroke
+			(width 0)
+			(type default)
+		)
+	)
+	(wire
+		(pts
+			(xy 40.64 101.6) (xy 59.69 101.6)
 		)
 		(stroke
@@
 	(wire
 		(pts
-			(xy 40.64 95.25) (xy 59.69 95.25)
-		)
-		(stroke
-			(width 0)
-			(type default)
-		)
-	)
-	(wire
-		(pts
-			(xy 40.64 80.01) (xy 59.69 80.01)
-		)
-		(stroke
-			(width 0)
-			(type default)
-		)
-	)
-	(wire
-		(pts
-			(xy 96.52 67.31) (xy 96.52 83.82)
-		)
-		(stroke
-			(width 0)
-			(type default)
-		)
-	)
-	(wire
-		(pts
-			(xy 96.52 83.82) (xy 92.71 83.82)
-		)
-		(stroke
-			(width 0)
-			(type default)
-		)
-	)
-	(wire
-		(pts
-			(xy 97.79 86.36) (xy 92.71 86.36)
-		)
-		(stroke
-			(width 0)
-			(type default)
-		)
-	)
-	(wire
-		(pts
-			(xy 97.79 57.15) (xy 92.71 57.15)
-		)
-		(stroke
-			(width 0)
-			(type default)
-		)
-	)
-	(wire
-		(pts
-			(xy 96.52 36.83) (xy 96.52 54.61)
-		)
-		(stroke
-			(width 0)
-			(type default)
-		)
-	)
-	(wire
-		(pts
-			(xy 92.71 36.83) (xy 96.52 36.83)
-		)
-		(stroke
-			(width 0)
-			(type default)
-		)
-	)
-	(wire
-		(pts
-			(xy 96.52 54.61) (xy 92.71 54.61)
+			(xy 40.64 119.38) (xy 59.69 119.38)
+		)
+		(stroke
+			(width 0)
+			(type default)
+		)
+	)
+	(wire
+		(pts
+			(xy 40.64 104.14) (xy 59.69 104.14)
+		)
+		(stroke
+			(width 0)
+			(type default)
+		)
+	)
+	(wire
+		(pts
+			(xy 97.79 54.61) (xy 92.71 54.61)
 		)
 		(stroke
@@
 	(wire
 		(pts
-			(xy 40.64 92.71) (xy 59.69 92.71)
-		)
-		(stroke
-			(width 0)
-			(type default)
-		)
-	)
-	(wire
-		(pts
-			(xy 92.71 64.77) (xy 97.79 64.77)
-		)
-		(stroke
-			(width 0)
-			(type default)
-		)
-	)
-	(wire
-		(pts
-			(xy 97.79 64.77) (xy 97.79 86.36)
-		)
-		(stroke
-			(width 0)
-			(type default)
-		)
-	)
-	(wire
-		(pts
-			(xy 40.64 97.79) (xy 59.69 97.79)
-		)
-		(stroke
-			(width 0)
-			(type default)
-		)
-	)
-	(wire
-		(pts
-			(xy 40.64 90.17) (xy 59.69 90.17)
-		)
-		(stroke
-			(width 0)
-			(type default)
-		)
-	)
-	(wire
-		(pts
-			(xy 97.79 34.29) (xy 97.79 57.15)
-		)
-		(stroke
-			(width 0)
-			(type default)
+			(xy 40.64 116.84) (xy 59.69 116.84)
+		)
+		(stroke
+			(width 0)
+			(type default)
+		)
+	)
+	(wire
+		(pts
+			(xy 40.64 121.92) (xy 59.69 121.92)
+		)
+		(stroke
+			(width 0)
+			(type default)
+		)
+	)
+	(wire
+		(pts
+			(xy 40.64 114.3) (xy 59.69 114.3)
+		)
+		(stroke
+			(width 0)
+			(type default)
+		)
+	)
+	(wire
+		(pts
+			(xy 97.79 36.83) (xy 97.79 54.61)
+		)
+		(stroke
+			(width 0)
+			(type default)
+		)
+	)
+	(sheet
+		(at 59.69 74.93)
+		(size 33.02 19.685)
+		(exclude_from_sim no)
+		(in_bom yes)
+		(on_board yes)
+		(dnp no)
+		(fields_autoplaced yes)
+		(stroke
+			(width 0.1524)
+			(type solid)
+		)
+		(fill
+			(color 0 0 0 0.0000)
+		)
+		(property "Sheetname" "inverter_self_osc_feedback_pass"
+			(at 59.69 74.2184 0)
+			(effects
+				(font
+					(size 1.27 1.27)
+				)
+				(justify left bottom)
+			)
+		)
+		(property "Sheetfile" "self_oscillation_feedback_pass.kicad_sch"
+			(at 59.69 95.1996 0)
+			(effects
+				(font
+					(size 1.27 1.27)
+				)
+				(justify left top)
+			)
+		)
+		(instances
+			(project "hardware"
+				(path "/606d342f-174b-4504-b335-50f65aa4e733/31b9362a-87aa-4ca5-9e9f-d5489b7d3e5d"
+					(page "15")
+				)
+			)
 		)
 	)
@@
 			)
 		)
-		(pin "INVERTER_RAW_FEEDBACK-" bidirectional
+		(pin "INVERTER_RAW_FEEDBACK+" bidirectional
 			(at 92.71 54.61 0)
 			(effects
@@
 			)
 		)
-		(pin "INVERTER_FEEDBACK+" bidirectional
-			(at 92.71 64.77 0)
-			(effects
-				(font
-					(size 1.27 1.27)
-				)
-				(justify right)
-			)
-		)
-		(pin "INVERTER_FEEDBACK-" bidirectional
+		(pin "INVERTER_RUN_STATE" bidirectional
 			(at 92.71 67.31 0)
-			(effects
-				(font
-					(size 1.27 1.27)
-				)
-				(justify right)
-			)
-		)
-		(pin "INVERTER_RAW_FEEDBACK+" bidirectional
-			(at 92.71 57.15 0)
 			(effects
 				(font
@@
 	(sheet
 		(at 20.955 27.94)
-		(size 19.685 71.755)
+		(size 19.685 97.155)
 		(exclude_from_sim no)
 		(in_bom yes)
@@
 		)
 		(property "Sheetfile" "input_supply.kicad_sch"
-			(at 20.955 100.2796 0)
+			(at 20.955 125.6796 0)
 			(effects
 				(font
@@
 		)
 		(pin "INVERTER_GDT_2A" bidirectional
-			(at 40.64 95.25 0)
+			(at 40.64 119.38 0)
 			(effects
 				(font
@@
 		)
 		(pin "INVERTER_GDT_1B" bidirectional
-			(at 40.64 92.71 0)
+			(at 40.64 116.84 0)
 			(effects
 				(font
@@
 		)
 		(pin "inverter_15v_a" bidirectional
-			(at 40.64 77.47 0)
+			(at 40.64 101.6 0)
 			(effects
 				(font
@@
 		)
 		(pin "INVERTER_GDT_1A" bidirectional
-			(at 40.64 90.17 0)
+			(at 40.64 114.3 0)
 			(effects
 				(font
@@
 		)
 		(pin "INVERTER_GDT_2B" bidirectional
-			(at 40.64 97.79 0)
+			(at 40.64 121.92 0)
 			(effects
 				(font
@@
 		)
 		(pin "inverter_15v_b" bidirectional
-			(at 40.64 80.01 0)
+			(at 40.64 104.14 0)
 			(effects
 				(font
@@
 	)
 	(sheet
-		(at 59.69 75.565)
+		(at 59.69 99.695)
 		(size 33.02 24.13)
 		(exclude_from_sim no)
@@
 		)
 		(property "Sheetname" "inverter_gdt_outstage"
-			(at 59.69 74.8534 0)
+			(at 59.69 98.9834 0)
 			(effects
 				(font
@@
 		)
 		(property "Sheetfile" "output_stage.kicad_sch"
-			(at 59.69 100.2796 0)
+			(at 59.69 124.4096 0)
 			(effects
 				(font
@@
 		)
 		(pin "INVERTER_GDT_1B" bidirectional
-			(at 59.69 92.71 180)
+			(at 59.69 116.84 180)
 			(effects
 				(font
@@
 		)
 		(pin "INVERTER_GDT_1A" bidirectional
-			(at 59.69 90.17 180)
+			(at 59.69 114.3 180)
 			(effects
 				(font
@@
 		)
 		(pin "inverter_15v_b" bidirectional
-			(at 59.69 80.01 180)
+			(at 59.69 104.14 180)
 			(effects
 				(font
@@
 		)
 		(pin "inverter_15v_a" bidirectional
-			(at 59.69 77.47 180)
+			(at 59.69 101.6 180)
 			(effects
 				(font
@@
 		)
 		(pin "INVERTER_GDT_2A" bidirectional
-			(at 59.69 95.25 180)
+			(at 59.69 119.38 180)
 			(effects
 				(font
@@
 		)
 		(pin "INVERTER_GDT_2B" bidirectional
-			(at 59.69 97.79 180)
+			(at 59.69 121.92 180)
 			(effects
 				(font
@@
 		)
 		(pin "INVERTER_FEEDBACK+" bidirectional
-			(at 92.71 86.36 0)
+			(at 92.71 110.49 0)
 			(effects
 				(font
@@
 		)
 		(pin "INVERTER_FEEDBACK-" bidirectional
-			(at 92.71 83.82 0)
+			(at 92.71 107.95 0)
 			(effects
 				(font
@@
 		)
 		(pin "INVERTER_RAW_FEEDBACK+" bidirectional
+			(at 92.71 36.83 0)
+			(effects
+				(font
+					(size 1.27 1.27)
+				)
+				(justify right)
+			)
+		)
+		(pin "INVERTER_RAW_FEEDBACK-" bidirectional
 			(at 92.71 34.29 0)
 			(effects
 				(font
-					(size 1.27 1.27)
-				)
-				(justify right)
-			)
-		)
-		(pin "INVERTER_RAW_FEEDBACK-" bidirectional
-			(at 92.71 36.83 0)
-			(effects
-				(font

Commit message: idk some changes
Other:
- removed sheet inverter_self_osc_feedback_pass
Changed lines of the file:
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@@
-	)
-	(sheet
-		(at 59.69 74.93)
-		(size 33.02 19.685)
-		(exclude_from_sim no)
-		(in_bom yes)
-		(on_board yes)
-		(dnp no)
-		(fields_autoplaced yes)
-		(stroke
-			(width 0.1524)
-			(type solid)
-		)
-		(fill
-			(color 0 0 0 0.0000)
-		)
-		(property "Sheetname" "inverter_self_osc_feedback_pass"
-			(at 59.69 74.2184 0)
-			(effects
-				(font
-					(size 1.27 1.27)
-				)
-				(justify left bottom)
-			)
-		)
-		(property "Sheetfile" "self_oscillation_feedback_pass.kicad_sch"
-			(at 59.69 95.1996 0)
-			(effects
-				(font
-					(size 1.27 1.27)
-				)
-				(justify left top)
-			)
-		)
-		(instances
-			(project "hardware"
-				(path "/606d342f-174b-4504-b335-50f65aa4e733/31b9362a-87aa-4ca5-9e9f-d5489b7d3e5d"
-					(page "15")
-				)
-			)
-		)
 	)
 	(sheet

Commit message: completed-ish inverter board, probably not, but anyway
Other:
- sheet interrupt_cross_off ports: added INVERTER_FEEDBACK+, INVERTER_FEEDBACK-, INVERTER_RAW_FEEDBACK-; removed INVERTER_RUN_STATE
- sheet inverter_gdt_outstage ports: added inverter_12v; removed inverter_15v_a, inverter_15v_b
- sheet inverter_input_supply ports: added inverter_12v; removed inverter_15v_a, inverter_15v_b
Changed lines of the file:
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@@
+	(wire
+		(pts
+			(xy 100.33 110.49) (xy 92.71 110.49)
+		)
+		(stroke
+			(width 0)
+			(type default)
+		)
+	)
 	(wire
 		(pts
@@
 	(wire
 		(pts
-			(xy 40.64 104.14) (xy 59.69 104.14)
+			(xy 100.33 34.29) (xy 92.71 34.29)
+		)
+		(stroke
+			(width 0)
+			(type default)
+		)
+	)
+	(wire
+		(pts
+			(xy 92.71 63.5) (xy 100.33 63.5)
 		)
 		(stroke
@@
 	(wire
 		(pts
+			(xy 92.71 66.04) (xy 97.79 66.04)
+		)
+		(stroke
+			(width 0)
+			(type default)
+		)
+	)
+	(wire
+		(pts
+			(xy 97.79 107.95) (xy 92.71 107.95)
+		)
+		(stroke
+			(width 0)
+			(type default)
+		)
+	)
+	(wire
+		(pts
 			(xy 40.64 30.48) (xy 59.69 30.48)
 		)
@@
 	(wire
 		(pts
+			(xy 92.71 57.15) (xy 100.33 57.15)
+		)
+		(stroke
+			(width 0)
+			(type default)
+		)
+	)
+	(wire
+		(pts
+			(xy 100.33 63.5) (xy 100.33 110.49)
+		)
+		(stroke
+			(width 0)
+			(type default)
+		)
+	)
+	(wire
+		(pts
+			(xy 97.79 66.04) (xy 97.79 107.95)
+		)
+		(stroke
+			(width 0)
+			(type default)
+		)
+	)
+	(wire
+		(pts
 			(xy 40.64 116.84) (xy 59.69 116.84)
+		)
+		(stroke
+			(width 0)
+			(type default)
+		)
+	)
+	(wire
+		(pts
+			(xy 100.33 57.15) (xy 100.33 34.29)
 		)
 		(stroke
@@
 			)
 		)
-		(pin "INVERTER_RUN_STATE" bidirectional
-			(at 92.71 67.31 0)
+		(pin "INVERTER_FEEDBACK+" bidirectional
+			(at 92.71 63.5 0)
+			(effects
+				(font
+					(size 1.27 1.27)
+				)
+				(justify right)
+			)
+		)
+		(pin "INVERTER_FEEDBACK-" bidirectional
+			(at 92.71 66.04 0)
+			(effects
+				(font
+					(size 1.27 1.27)
+				)
+				(justify right)
+			)
+		)
+		(pin "INVERTER_RAW_FEEDBACK-" bidirectional
+			(at 92.71 57.15 0)
 			(effects
 				(font
@@
 			)
 		)
-		(pin "inverter_15v_a" bidirectional
-			(at 40.64 101.6 0)
-			(effects
-				(font
-					(size 1.27 1.27)
-				)
-				(justify right)
-			)
-		)
 		(pin "INVERTER_GDT_1A" bidirectional
 			(at 40.64 114.3 0)
@@
 			)
 		)
-		(pin "inverter_15v_b" bidirectional
-			(at 40.64 104.14 0)
+		(pin "inverter_12v" bidirectional
+			(at 40.64 101.6 0)
 			(effects
 				(font
@@
 			)
 		)
-		(pin "inverter_15v_b" bidirectional
-			(at 59.69 104.14 180)
-			(effects
-				(font
-					(size 1.27 1.27)
-				)
-				(justify left)
-			)
-		)
-		(pin "inverter_15v_a" bidirectional
-			(at 59.69 101.6 180)
-			(effects
-				(font
-					(size 1.27 1.27)
-				)
-				(justify left)
-			)
-		)
 		(pin "INVERTER_GDT_2A" bidirectional
 			(at 59.69 119.38 180)
@@
 			)
 		)
+		(pin "inverter_12v" bidirectional
+			(at 59.69 101.6 180)
+			(effects
+				(font
+					(size 1.27 1.27)
+				)
+				(justify left)
+			)
+		)

Commit message: minor changes
Changed lines of the file:
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@@
 	(wire
 		(pts
-			(xy 40.64 101.6) (xy 59.69 101.6)
+			(xy 40.64 78.74) (xy 59.69 78.74)
 		)
 		(stroke
@@
 	(wire
 		(pts
-			(xy 100.33 110.49) (xy 92.71 110.49)
-		)
-		(stroke
-			(width 0)
-			(type default)
-		)
-	)
-	(wire
-		(pts
-			(xy 40.64 119.38) (xy 59.69 119.38)
+			(xy 100.33 87.63) (xy 92.71 87.63)
+		)
+		(stroke
+			(width 0)
+			(type default)
+		)
+	)
+	(wire
+		(pts
+			(xy 40.64 96.52) (xy 59.69 96.52)
 		)
 		(stroke
@@
 	(wire
 		(pts
-			(xy 97.79 107.95) (xy 92.71 107.95)
+			(xy 97.79 85.09) (xy 92.71 85.09)
 		)
 		(stroke
@@
 	(wire
 		(pts
-			(xy 100.33 63.5) (xy 100.33 110.49)
-		)
-		(stroke
-			(width 0)
-			(type default)
-		)
-	)
-	(wire
-		(pts
-			(xy 97.79 66.04) (xy 97.79 107.95)
-		)
-		(stroke
-			(width 0)
-			(type default)
-		)
-	)
-	(wire
-		(pts
-			(xy 40.64 116.84) (xy 59.69 116.84)
+			(xy 100.33 63.5) (xy 100.33 87.63)
+		)
+		(stroke
+			(width 0)
+			(type default)
+		)
+	)
+	(wire
+		(pts
+			(xy 97.79 66.04) (xy 97.79 85.09)
+		)
+		(stroke
+			(width 0)
+			(type default)
+		)
+	)
+	(wire
+		(pts
+			(xy 40.64 93.98) (xy 59.69 93.98)
 		)
 		(stroke
@@
 	(wire
 		(pts
-			(xy 40.64 121.92) (xy 59.69 121.92)
-		)
-		(stroke
-			(width 0)
-			(type default)
-		)
-	)
-	(wire
-		(pts
-			(xy 40.64 114.3) (xy 59.69 114.3)
+			(xy 40.64 99.06) (xy 59.69 99.06)
+		)
+		(stroke
+			(width 0)
+			(type default)
+		)
+	)
+	(wire
+		(pts
+			(xy 40.64 91.44) (xy 59.69 91.44)
 		)
 		(stroke
@@
 	(sheet
 		(at 20.955 27.94)
-		(size 19.685 97.155)
+		(size 19.685 73.66)
 		(exclude_from_sim no)
 		(in_bom yes)
@@
 		)
 		(property "Sheetfile" "input_supply.kicad_sch"
-			(at 20.955 125.6796 0)
+			(at 20.955 102.1846 0)
 			(effects
 				(font
@@
 		)
 		(pin "INVERTER_GDT_2A" bidirectional
-			(at 40.64 119.38 0)
+			(at 40.64 96.52 0)
 			(effects
 				(font
@@
 		)
 		(pin "INVERTER_GDT_1B" bidirectional
-			(at 40.64 116.84 0)
+			(at 40.64 93.98 0)
 			(effects
 				(font
@@
 		)
 		(pin "INVERTER_GDT_1A" bidirectional
-			(at 40.64 114.3 0)
+			(at 40.64 91.44 0)
 			(effects
 				(font
@@
 		)
 		(pin "INVERTER_GDT_2B" bidirectional
-			(at 40.64 121.92 0)
+			(at 40.64 99.06 0)
 			(effects
 				(font
@@
 		)
 		(pin "inverter_12v" bidirectional
-			(at 40.64 101.6 0)
+			(at 40.64 78.74 0)
 			(effects
 				(font
@@
 	)
 	(sheet
-		(at 59.69 99.695)
+		(at 59.69 76.835)
 		(size 33.02 24.13)
 		(exclude_from_sim no)
@@
 		)
 		(property "Sheetname" "inverter_gdt_outstage"
-			(at 59.69 98.9834 0)
+			(at 59.69 76.1234 0)
 			(effects
 				(font
@@
 		)
 		(property "Sheetfile" "output_stage.kicad_sch"
-			(at 59.69 124.4096 0)
+			(at 59.69 101.5496 0)
 			(effects
 				(font
@@
 		)
 		(pin "INVERTER_GDT_1B" bidirectional
-			(at 59.69 116.84 180)
+			(at 59.69 93.98 180)
 			(effects
 				(font
@@
 		)
 		(pin "INVERTER_GDT_1A" bidirectional
-			(at 59.69 114.3 180)
+			(at 59.69 91.44 180)
 			(effects
 				(font
@@
 		)
 		(pin "INVERTER_GDT_2A" bidirectional
-			(at 59.69 119.38 180)
+			(at 59.69 96.52 180)
 			(effects
 				(font
@@
 		)
 		(pin "INVERTER_GDT_2B" bidirectional
-			(at 59.69 121.92 180)
+			(at 59.69 99.06 180)
 			(effects
 				(font
@@
 		)
 		(pin "INVERTER_FEEDBACK+" bidirectional
-			(at 92.71 110.49 0)
+			(at 92.71 87.63 0)
 			(effects
 				(font
@@
 		)
 		(pin "INVERTER_FEEDBACK-" bidirectional
-			(at 92.71 107.95 0)
+			(at 92.71 85.09 0)
 			(effects
 				(font
@@
 		)
 		(pin "inverter_12v" bidirectional
-			(at 59.69 101.6 180)
-			(effects
-				(font
+			(at 59.69 78.74 180)
+			(effects
+				(font
