File: hardware/control/inverter/output_stage.kicad_sch (KiCad schematic)
At the start: 0 parts

Commit message: completed-ish inverter board, probably not, but anyway
Parts:
- added C26, C32, C33, C36: 100n, symbol Device:C
- added C37, C39: 1u, symbol Device:C
- added C38, C40: 5u, symbol Device:C
- added C41, C42, C43, C44: 4.7u, symbol Device:C
- added D18, D19, D20, D22: 1N4148, PCM_Diode_THT_AKL:D_DO-35_SOD27_P7.62mm_Horizontal, symbol PCM_Diode_AKL:1N4148
- added J9: PINHD_2x4_Male, Connector_PinHeader_2.54mm:PinHeader_2x04_P2.54mm_Vertical, symbol PCM_SL_Pin_Headers:PINHD_2x4_Male
- added Q2, Q3, Q4, Q5: AOD609, PCM_Package_TO_SOT_SMD_AKL:TO-252-4, symbol PCM_Transistor_MOSFET_AKL:AOD609
- added R15, R19, R23, R24: 1k, symbol Device:R
- added U21, U22: TC4427xOA, Package_SO:SOIC-8_3.9x4.9mm_P1.27mm, symbol Driver_FET:TC4427xOA
Connections:
- net INVERTER_FEEDBACK+: now also J9.1, J9.3
- net INVERTER_FEEDBACK-: now also J9.5, J9.7
- net INVERTER_GDT_1A: now also Q2.3 (C)
- net INVERTER_GDT_1B: now also Q3.3 (C)
- net INVERTER_GDT_2A: now also Q4.3 (C)
- net INVERTER_GDT_2B: now also Q5.3 (C)
- new net: C26.1, D18.2 (A), Q3.5 (G2), R15.2
- new net: C33.1, D22.2 (A), Q2.5 (G2), R19.2
- new net: C32.1, D19.2 (A), Q4.5 (G2), R23.2
- new net: C32.2, Q4.2 (G1), U22.7 (OUT_A)
- new net: C33.2, Q2.2 (G1), U21.7 (OUT_A)
- new net: J9.2, J9.8, U21.2 (IN_A), U22.2 (IN_A)
- new net: J9.4, J9.6, U21.4 (IN_B), U22.4 (IN_B)
- new net: C26.2, Q3.2 (G1), U21.5 (OUT_B)
- new net: C36.2, Q5.2 (G1), U22.5 (OUT_B)
- new net: C36.1, D20.2 (A), Q5.5 (G2), R24.2
- new net GND: C37.2, C38.2, C39.2, C40.2, C41.1, C42.1, C43.1, C44.1, Q2.1 (S1), Q3.1 (S1), Q4.1 (S1), Q5.1 (S1), U21.3 (GND), U22.3 (GND)
- new net bus_24V: C41.2, C42.2, C43.2, C44.2, D18.1 (K), D19.1 (K), D20.1 (K), D22.1 (K), Q2.4 (S2), Q3.4 (S2), Q4.4 (S2), Q5.4 (S2), R15.1, R19.1, R23.1, R24.1
- new net inverter_12v: C37.1, C38.1, C39.1, C40.1, U21.6 (V_{DD}), U22.6 (V_{DD})

Commit message: minor changes
Parts:
- added C45, C46: 2.2u, symbol Device:C
Connections:
- net INVERTER_GDT_1B: now also C45.2; no longer Q3.3 (C)
- net INVERTER_GDT_2B: now also C46.2; no longer Q5.3 (C)
- new net: C46.1, Q5.3 (C)
- new net: C45.1, Q3.3 (C)
Changed lines of the file:
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@@
 	(wire
 		(pts
+			(xy 191.77 130.81) (xy 193.04 130.81)
+		)
+		(stroke
+			(width 0)
+			(type default)
+		)
+	)
+	(wire
+		(pts
 			(xy 143.51 114.3) (xy 163.83 114.3)
 		)
@@
 	(wire
 		(pts
+			(xy 182.88 82.55) (xy 184.15 82.55)
+		)
+		(stroke
+			(width 0)
+			(type default)
+		)
+	)
+	(wire
+		(pts
 			(xy 102.87 77.47) (xy 100.33 77.47)
 		)
@@
 	(wire
 		(pts
-			(xy 182.88 130.81) (xy 182.88 133.35)
-		)
-		(stroke
-			(width 0)
-			(type default)
-		)
-	)
-	(wire
-		(pts
 			(xy 143.51 113.03) (xy 143.51 114.3)
 		)
@@
 	(wire
 		(pts
+			(xy 191.77 82.55) (xy 193.04 82.55)
+		)
+		(stroke
+			(width 0)
+			(type default)
+		)
+	)
+	(wire
+		(pts
 			(xy 113.03 97.79) (xy 166.37 97.79)
 		)
@@
 	(wire
 		(pts
+			(xy 182.88 130.81) (xy 184.15 130.81)
+		)
+		(stroke
+			(width 0)
+			(type default)
+		)
+	)
+	(wire
+		(pts
 			(xy 102.87 132.08) (xy 104.14 132.08)
 		)
@@
 	(wire
 		(pts
-			(xy 182.88 82.55) (xy 182.88 86.36)
-		)
-		(stroke
-			(width 0)
-			(type default)
-		)
-	)
-	(wire
-		(pts
 			(xy 115.57 125.73) (xy 115.57 127)
 		)
@@
 	(hierarchical_label "INVERTER_GDT_2B"
 		(shape bidirectional)
-		(at 182.88 133.35 0)
+		(at 193.04 130.81 0)
 		(effects
 			(font
@@
 	(hierarchical_label "INVERTER_GDT_1B"
 		(shape bidirectional)
-		(at 182.88 86.36 0)
+		(at 193.04 82.55 0)
 		(effects
 			(font
@@
 		(dnp no)
 		(property "Reference" "Q4"
-			(at 147.574 124.206 0)
+			(at 147.066 118.872 0)
 			(effects
 				(font
@@
 		)
 		(property "Value" "AOD609"
-			(at 149.352 127 0)
+			(at 148.844 121.666 0)
 			(effects
 				(font
@@
 		(on_board yes)
 		(dnp no)
-		(fields_autoplaced yes)
 		(property "Reference" "Q5"
-			(at 185.42 124.3898 0)
+			(at 182.88 119.634 0)
 			(effects
 				(font
@@
 		)
 		(property "Value" "AOD609"
-			(at 185.42 126.9298 0)
+			(at 183.896 121.92 0)
 			(effects
 				(font
@@
 	)
 	(symbol
+		(lib_id "Device:C")
+		(at 187.96 130.81 90)
+		(unit 1)
+		(exclude_from_sim no)
+		(in_bom yes)
+		(on_board yes)
+		(dnp no)
+		(property "Reference" "C46"
+			(at 187.96 125.476 90)
+			(effects
+				(font
+					(size 1.27 1.27)
+				)
+			)
+		)
+		(property "Value" "2.2u"
+			(at 188.214 127.508 90)
+			(effects
+				(font
+					(size 1.27 1.27)
+				)
+			)
+		)
+		(property "Footprint" ""
+			(at 191.77 129.8448 0)
+			(effects
+				(font
+					(size 1.27 1.27)
+				)
+				(hide yes)
+			)
+		)
+		(property "Datasheet" "~"
+			(at 187.96 130.81 0)
+			(effects
+				(font
+					(size 1.27 1.27)
+				)
+				(hide yes)
+			)
+		)
+		(property "Description" "Unpolarized capacitor"
+			(at 187.96 130.81 0)
+			(effects
+				(font
+					(size 1.27 1.27)
+				)
+				(hide yes)
+			)
+		)
+		(pin "2"
+		)
+		(pin "1"
+		)
+		(instances
+			(project "hardware"
+				(path "/606d342f-174b-4504-b335-50f65aa4e733/31b9362a-87aa-4ca5-9e9f-d5489b7d3e5d/a4b4d7e4-1905-4659-a585-0a112bd7ab50"
+					(reference "C46")
+					(unit 1)
+				)
+			)
+		)
+	)
+	(symbol
 		(lib_id "power:GND")
 		(at 143.51 57.15 180)
@@
 		(on_board yes)
 		(dnp no)
-		(fields_autoplaced yes)
 		(property "Reference" "Q3"
-			(at 185.42 76.1298 0)
+			(at 182.372 71.12 0)
 			(effects
 				(font
@@
 		)
 		(property "Value" "AOD609"
-			(at 185.42 78.6698 0)
+			(at 183.896 73.406 0)
 			(effects
 				(font
@@
 	)
 	(symbol
+		(lib_id "Device:C")
+		(at 187.96 82.55 90)
+		(unit 1)
+		(exclude_from_sim no)
+		(in_bom yes)
+		(on_board yes)
+		(dnp no)
+		(property "Reference" "C45"
+			(at 187.96 77.216 90)
+			(effects
+				(font
+					(size 1.27 1.27)
+				)
+			)
+		)
+		(property "Value" "2.2u"
+			(at 188.214 79.248 90)
+			(effects
+				(font
+					(size 1.27 1.27)
+				)
+			)
+		)
+		(property "Footprint" ""
+			(at 191.77 81.5848 0)
+			(effects
+				(font
+					(size 1.27 1.27)
+				)
+				(hide yes)
+			)
+		)
+		(property "Datasheet" "~"
+			(at 187.96 82.55 0)
+			(effects
+				(font
+					(size 1.27 1.27)
+				)
+				(hide yes)
+			)
+		)
+		(property "Description" "Unpolarized capacitor"
+			(at 187.96 82.55 0)
+			(effects
+				(font
+					(size 1.27 1.27)
+				)
+				(hide yes)
+			)
+		)
+		(pin "2"
+		)
+		(pin "1"
+		)
+		(instances
+			(project ""
+				(path "/606d342f-174b-4504-b335-50f65aa4e733/31b9362a-87aa-4ca5-9e9f-d5489b7d3e5d/a4b4d7e4-1905-4659-a585-0a112bd7ab50"
+					(reference "C45")
+					(unit 1)
+				)
+			)
+		)
+	)
+	(symbol
 		(lib_id "PCM_Diode_AKL:1N4148")
 		(at 128.27 119.38 90)
@@
 		(dnp no)
 		(property "Reference" "Q2"
-			(at 147.574 75.946 0)
+			(at 147.066 70.612 0)
 			(effects
 				(font
@@
 		)
 		(property "Value" "AOD609"
-			(at 149.352 78.74 0)
+			(at 148.844 73.406 0)
 			(effects
 				(font
